File: structure_board.kicad_sch (KiCad schematic)
At the start: 19 parts

Commit message: cleanup and export 3d-models
Connections:
- no-connect marks 19 -> 18
Other:
- company: (none) -> TUDSaT
- title: (none) -> Structure board
- moved on the sheet: H1, H10, H11, H12, H13, H14, H15, H2, H20, H21, H22, H23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
